File: OpenServo/V4-EDA-preliminary-work/OSv4_H-bridge.sch (KiCad schematic (older format))
At the start: 18 parts, among them M1 CONN_1, M2 CONN_1, M3 CONN_1, Q1 NP_MOSFET, Q4 NP_MOSFET, U1 ZXCT1009, U5 TC4428A, U6 TC4428A

Commit message: no message
Parts:
- renumbered Q1 to U7, Q4 to U8
Changed lines of the file:
@@
-EESchema Schematic File Version 2  date 25/04/2010 17:16:50
+EESchema Schematic File Version 2  date 04/05/2010 11:09:49
 LIBS:power
 LIBS:device
@@
 Sheet 3 3
 Title "OpenServo v4 preliminary work-up, © OpenServo project 2010"
-Date "25 apr 2010"
+Date "4 may 2010"
 Rev "0.0"
 Comp ""
@@
 Potential MOSFETs for Q1/Q4:\nSP8M4\nFDS8858CZ\nFDS9934C??
 $Comp
-L NP_MOSFET Q4
+L NP_MOSFET U8
 U 2 1 4BAFC8F5
 P 6450 4200
-F 0 "Q4" H 6225 4365 60  0000 C CNN
+F 0 "U8" H 6225 4365 60  0000 C CNN
 F 1 "NP_MOSFET" H 6100 4500 60  0000 C CNN
 F 2 "SO8E" H 6165 4425 60  0001 C CNN
@@
 $EndComp
 $Comp
-L NP_MOSFET Q4
+L NP_MOSFET U8
 U 1 1 4BAFC8A1
 P 6450 5800
-F 0 "Q4" H 6225 5965 60  0000 C CNN
+F 0 "U8" H 6225 5965 60  0000 C CNN
 F 1 "NP_MOSFET" H 6100 6100 60  0000 C CNN
 F 2 "SO8E" H 6165 6025 60  0001 C CNN
@@
 $EndComp
 $Comp
-L NP_MOSFET Q1
+L NP_MOSFET U7
 U 2 1 4BAFC7E3
 P 5150 4200
-F 0 "Q1" H 4925 4365 60  0000 C CNN
+F 0 "U7" H 4925 4365 60  0000 C CNN
 F 1 "NP_MOSFET" H 4800 4500 60  0000 C CNN
 F 2 "SO8E" H 5150 4200 60  0001 C CNN
@@
 $EndComp
 $Comp
-L NP_MOSFET Q1
+L NP_MOSFET U7
 U 1 1 4BAFC774
 P 5150 5800
-F 0 "Q1" H 4925 5965 60  0000 C CNN
+F 0 "U7" H 4925 5965 60  0000 C CNN
 F 1 "NP_MOSFET" H 4800 6100 60  0000 C CNN
 F 2 "SO8E" H 4865 6025 60  0001 C CNN

Commit message: no message
Parts:
- C1, C2: Comments (none) -> X5R, ±10%, 16V, Ceramic; Farnell (none) -> 1735530; Manufacturer (none) -> muRata; Mfg. P/N (none) -> GRM21BR61E106KA73L
- C3: footprint SM0402 -> SM0603; Comments (none) -> X5R, ±10%, 16V, Ceramic
- C4, C5: Comments (none) -> X7R, ±10%, 16V, Ceramic; Farnell (none) -> 1758896; Manufacturer (none) -> multicomp; Mfg. P/N (none) -> MCCA000050
- D2: value ZENER -> 3.6V; footprint SM0402 -> SOD-123; Comments (none) -> 3.6V, 0.5W, 5%; Farnell (none) -> 1700854; Manufacturer (none) -> Fairchild Semiconductor; Mfg. P/N (none) -> MMSZ5227B
- R2: Comments (none) -> 0.25W, 2%, current sense; Farnell (none) -> 9376771; Manufacturer (none) -> Susumu; Mfg. P/N (none) -> RL1220T-R050-G
- RP2: Farnell (none) -> 1770152RL; Manufacturer (none) -> Bourns; Mfg. P/N (none) -> CAY10-103J4LF
- U1: footprint SOT23_3 -> SOT23-3
- U5, U6: footprint MSOP_8 -> SOIC8; Farnell (none) -> 1332312; Manufacturer (none) -> Microchip; Mfg. P/N (none) -> TC4428ACOA
- U7, U8: footprint SO8E -> SOIC8
Connections:
- net EN_A: now also RP2.5 (R4); no longer RP2.6 (R3)
- net EN_B: now also RP2.1 (P1); no longer RP2.7 (R2)
- net GND: now also RP2.6 (R3), RP2.8 (R1); no longer RP2.1 (P1), RP2.3 (P3)
- net PWM_A: now also RP2.3 (P3); no longer RP2.5 (R4)
- net PWM_B: now also RP2.7 (R2); no longer RP2.8 (R1)
Other:
- note added: "Potential MOSFETs for U7 & U8:\nSP8M4\nFDS8858CZ\nFDS9934C??"
- note added: "TODO: Change R2 for 0.5W 1% SM1206?"
- note removed: "Potential MOSFETs for Q1/Q4:\nSP8M4\nFDS8858CZ\nFDS9934C??"
- note removed: "TODO: Do we need to\nReinstate R9, R10, R13\nand R14? If yes, then\nthey should be an\nRPACK to save\nPCB space.\n\nTODO: What value is needed\nfor the protection diode D2?\n"

Commit message: no message
Parts:
- C1, C2: Comments X5R, ±10%, 16V, Ceramic -> X5R, ±10%, 25V, Ceramic
- C3: Farnell (none) -> 1759407; Manufacturer (none) -> multicomp; Mfg. P/N (none) -> MCCA000529
- RP2: footprint RP0804 -> CAY10-XXXJ4
- U1: Comments (none) -> Farnell equiv: 1132757; DigiKey (none) -> ZXCT1009FCT-ND; Farnell (none) -> See comments; Manufacturer (none) -> Zetex; Mfg. P/N (none) -> ZXCT1009FTA
Changed lines of the file:
@@
-EESchema Schematic File Version 2  date 07/05/2010 17:07:47
+EESchema Schematic File Version 2  date 08/05/2010 00:59:33
 LIBS:power
 LIBS:device
@@
 F 0 "RP2" H 2800 6700 40  0000 C CNN
 F 1 "R_PACK4" H 2800 6200 40  0000 C CNN
-F 2 "RP0804" H 2760 6740 60  0001 C CNN
+F 2 "CAY10-XXXJ4" H 2760 6740 60  0001 C CNN
 F 4 "Bourns" H 2800 6250 60  0001 C CNN "Manufacturer"
 F 5 "CAY10-103J4LF" H 2800 6250 60  0001 C CNN "Mfg. P/N"
@@
 F 1 "1uF" H 6950 1700 50  0000 L CNN
 F 2 "SM0603" H 7000 1950 60  0001 C CNN
-F 4 "" H 6900 1800 60  0001 C CNN "Manufacturer"
-F 5 "" H 6900 1800 60  0001 C CNN "Mfg. P/N"
-F 6 "" H 6900 1800 60  0001 C CNN "Farnell"
+F 4 "multicomp" H 6900 1800 60  0001 C CNN "Manufacturer"
+F 5 "MCCA000529" H 6900 1800 60  0001 C CNN "Mfg. P/N"
+F 6 "1759407" H 6900 1800 60  0001 C CNN "Farnell"
 F 7 "" H 6900 1800 60  0001 C CNN "DigiKey"
 F 8 "X5R, ±10%, 16V, Ceramic" H 6900 1800 60  0001 C CNN "Comments"
@@
 F 6 "1735530" H 6550 1800 60  0001 C CNN "Farnell"
 F 7 "" H 6550 1800 60  0001 C CNN "DigiKey"
-F 8 "X5R, ±10%, 16V, Ceramic" H 6550 1800 60  0001 C CNN "Comments"
+F 8 "X5R, ±10%, 25V, Ceramic" H 6550 1800 60  0001 C CNN "Comments"
 	1    6550 1800
 	1    0    0    -1
@@
 F 6 "1735530" H 6200 1800 60  0001 C CNN "Farnell"
 F 7 "" H 6200 1800 60  0001 C CNN "DigiKey"
-F 8 "X5R, ±10%, 16V, Ceramic" H 6200 1800 60  0001 C CNN "Comments"
+F 8 "X5R, ±10%, 25V, Ceramic" H 6200 1800 60  0001 C CNN "Comments"
 	1    6200 1800
 	1    0    0    -1
@@
 F 1 "ZXCT1009" V 5600 1550 60  0000 L CNN
 F 2 "SOT23-3" V 4890 1590 60  0001 C CNN
+F 4 "Zetex" H 5300 1800 60  0001 C CNN "Manufacturer"
+F 5 "ZXCT1009FTA" H 5300 1800 60  0001 C CNN "Mfg. P/N"
+F 6 "See comments" H 5300 1800 60  0001 C CNN "Farnell"
+F 7 "ZXCT1009FCT-ND" H 5300 1800 60  0001 C CNN "DigiKey"
+F 8 "Farnell equiv: 1132757" H 5300 1800 60  0001 C CNN "Comments"
 	1    5300 1800
 	0    1    1    0

Commit message: no message
Parts:
- U7, U8: value NP_MOSFET -> MOSFET; Farnell (none) -> 1525587; Manufacturer (none) -> ROHM; Mfg. P/N (none) -> SP8M4FU6TB
Connections:
- net EN_B: now also RP2.2 (P2); no longer RP2.1 (P1)
- net GND: now also RP2.3 (P3), RP2.7 (R2); no longer RP2.2 (P2), RP2.6 (R3)
- net PWM_A: now also RP2.1 (P1); no longer RP2.3 (P3)
- net PWM_B: now also RP2.6 (R3); no longer RP2.7 (R2)
- net at U5.5 (NC): now also U5.8 (OUT_B), U7.2 (G)
- no-connect marks 4 -> 3
Other:
- note added: "NOTE: According to the docs, pin 5 on U5 has\n"no internal connection"; it has been used for\nrouting purposes on the PCB.\n\nTODO: TEST!"
- note added: "U5 & U6 (TC4428A): Originally the intention was to use the\nMSOP-8 package which would allow more room on the PCB\nfor other things. However, this packaging only appears to be\navailable when purchased in large quantities; which is not\nworkable for a project where there is an expectation to be\nable to produce low-count runs."
Changed lines of the file:
@@
-EESchema Schematic File Version 2  date 08/05/2010 00:59:33
+EESchema Schematic File Version 2  date 08/05/2010 23:36:58
 LIBS:power
 LIBS:device
@@
 Sheet 3 3
 Title "OpenServo v4 preliminary work-up, © OpenServo project 2010"
-Date "7 may 2010"
+Date "8 may 2010"
 Rev "0.0"
 Comp ""
@@
 Comment4 ""
 $EndDescr
-Text Notes 5200 2550 0    60   ~ 0
-TODO: Change R2 for 0.5W 1% SM1206?
-Connection ~ 1800 4850
-Wire Wire Line
-	1800 4850 1800 6100
+Wire Wire Line
+	3350 7000 3350 6200
+Wire Wire Line
+	1800 6000 1800 5250
+Wire Wire Line
+	1800 6000 2600 6000
+Connection ~ 3900 5250
+Wire Wire Line
+	3900 4650 3900 5250
+Wire Wire Line
+	3900 4650 3800 4650
+Connection ~ 3200 6000
+Wire Wire Line
+	3000 6000 3200 6000
+Connection ~ 2050 6200
+Wire Wire Line
+	2600 6200 2050 6200
+Wire Wire Line
+	9950 6850 3500 6850
+Connection ~ 1600 4850
+Connection ~ 1800 5250
 Connection ~ 9950 4850
 Wire Wire Line
-	9950 4850 9950 6850
-Wire Wire Line
-	9950 6850 3750 6850
-Wire Wire Line
-	3750 6850 3750 6000
-Wire Wire Line
-	3750 6000 3000 6000
-Connection ~ 2400 6200
-Wire Wire Line
-	2600 6200 2400 6200
-Wire Wire Line
-	2400 6550 2400 6000
-Wire Wire Line
-	2400 6000 2600 6000
+	9950 6850 9950 4850
 Wire Wire Line
 	4900 5800 4200 5800
@@
 	6700 4200 7450 4200
 Wire Wire Line
-	6450 6000 6450 6200
+	6450 6200 6450 6000
 Connection ~ 6400 4550
 Wire Wire Line
-	6500 4450 6500 4550
+	6500 4550 6500 4450
 Wire Wire Line
 	6500 4550 6350 4550
@@
 	5100 5450 5100 5550
 Wire Wire Line
-	5150 6000 5150 6200
-Wire Wire Line
-	5100 4450 5100 4550
+	5150 6200 5150 6000
+Wire Wire Line
+	5100 4550 5100 4450
 Wire Wire Line
 	7850 5250 7450 5250
@@
 	4200 5250 4200 5800
 Wire Wire Line
-	3800 2300 3800 2400
+	3800 2400 3800 2300
 Wire Wire Line
 	3800 2400 4400 2400
@@
 	6550 2100 6550 2000
 Wire Wire Line
-	7250 2000 7250 2100
+	7250 2100 7250 2000
 Connection ~ 6900 1500
 Wire Wire Line
@@
 Connection ~ 3800 1800
 Wire Wire Line
-	7250 2100 6200 2100
+	6200 2100 7250 2100
 Connection ~ 5200 5000
 Wire Wire Line
@@
 	5100 4550 5250 4550
 Wire Wire Line
-	5200 4550 5200 5450
+	5200 5450 5200 4550
 Connection ~ 5800 6200
 Wire Wire Line
-	5150 6200 6450 6200
+	6450 6200 5150 6200
 Wire Wire Line
 	5150 3800 6450 3800
@@
 Connection ~ 6400 5000
 Wire Wire Line
-	5800 1500 7250 1500
+	7250 1500 5800 1500
 Wire Wire Line
 	5800 1400 5450 1400
@@
 Connection ~ 6900 2100
 Wire Wire Line
-	5800 2050 5800 3800
+	5800 3800 5800 2050
 Wire Wire Line
 	5800 1550 5800 1300
@@
 	4250 2500 4250 2400
 Wire Wire Line
-	3800 1900 3800 1800
+	3800 1800 3800 1900
 Wire Wire Line
 	4200 4850 4200 4200
@@
 	4000 3600 4000 5050
 Wire Wire Line
-	1200 4850 2300 4850
+	2300 4850 1200 4850
 Wire Wire Line
 	4000 5050 3800 5050
@@
 	6450 3800 6450 4000
 Wire Wire Line
-	6350 5550 6350 5450
+	6350 5450 6350 5550
 Wire Wire Line
 	6350 5450 6500 5450
@@
 	4200 4200 4900 4200
 Wire Wire Line
-	3000 6100 3200 6100
-Wire Wire Line
-	2600 5900 1600 5900
-Wire Wire Line
-	1600 5900 1600 5250
-Connection ~ 1600 5250
-Wire Wire Line
-	1800 6100 2600 6100
-Wire Wire Line
-	3000 5900 3200 5900
-Wire Wire Line
-	3200 5900 3200 6550
-Connection ~ 3200 6100
-Wire Wire Line
-	3000 6200 3600 6200
-Wire Wire Line
-	3600 6200 3600 7000
-Wire Wire Line
-	3600 7000 10100 7000
+	3200 5900 3000 5900
+Wire Wire Line
+	3200 6550 3200 5900
+Wire Wire Line
+	3350 7000 10100 7000
 Wire Wire Line
 	10100 7000 10100 5250
 Connection ~ 10100 5250
+Wire Wire Line
+	2600 6100 2050 6100
+Connection ~ 2050 6100
+Wire Wire Line
+	3350 6200 3000 6200
+Wire Wire Line
+	3000 6100 3500 6100
+Wire Wire Line
+	2600 5900 1600 5900
+Wire Wire Line
+	1600 5900 1600 4850
+Wire Wire Line
+	3500 6100 3500 6850
+Connection ~ 3500 6850
+Text Notes 1350 4200 0    60   ~ 0
+NOTE: According to the docs, pin 5 on U5 has\n"no internal connection"; it has been used for\nrouting purposes on the PCB.\n\nTODO: TEST!
+Text Notes 900  2650 0    60   ~ 0
+U5 & U6 (TC4428A): Originally the intention was to use the\nMSOP-8 package which would allow more room on the PCB\nfor other things. However, this packaging only appears to be\navailable when purchased in large quantities; which is not\nworkable for a project where there is an expectation to be\nable to produce low-count runs.
+Text Notes 5200 2550 0    60   ~ 0
+TODO: Change R2 for 0.5W 1% SM1206?
 $Comp
 L GND #PWR022
@@
 Text Notes 600  800  0    157  ~ 31
 NOTE: This is a Work In Progress; implement at your own risk.
-$Comp
-L GND #PWR023
-U 1 1 4BB67093
-P 2400 6550
-F 0 "#PWR023" H 2400 6550 30  0001 C CNN
-F 1 "GND" H 2400 6480 30  0001 C CNN
-	1    2400 6550
-	1    0    0    -1
-$EndComp
 $Comp
 L R_PACK4 RP2
@@
 P 6450 4200
 F 0 "U8" H 6225 4365 60  0000 C CNN
-F 1 "NP_MOSFET" H 6100 4500 60  0000 C CNN
+F 1 "MOSFET" H 6100 4500 60  0000 C CNN
 F 2 "SOIC8" H 6165 4425 60  0001 C CNN
+F 4 "ROHM" H 6450 4200 60  0001 C CNN "Manufacturer"
+F 5 "SP8M4FU6TB" H 6450 4200 60  0001 C CNN "Mfg. P/N"
+F 6 "1525587" H 6450 4200 60  0001 C CNN "Farnell"
+F 7 "" H 6450 4200 60  0001 C CNN "DigiKey"
+F 8 "" H 6450 4200 60  0001 C CNN "Comments"
 	2    6450 4200
 	-1   0    0    1
@@
 P 6450 5800
 F 0 "U8" H 6225 5965 60  0000 C CNN
-F 1 "NP_MOSFET" H 6100 6100 60  0000 C CNN
+F 1 "MOSFET" H 6100 6100 60  0000 C CNN
 F 2 "SOIC8" H 6165 6025 60  0001 C CNN
+F 4 "ROHM" H 6450 5800 60  0001 C CNN "Manufacturer"
+F 5 "SP8M4FU6TB" H 6450 5800 60  0001 C CNN "Mfg. P/N"
+F 6 "1525587" H 6450 5800 60  0001 C CNN "Farnell"
+F 7 "" H 6450 5800 60  0001 C CNN "DigiKey"
+F 8 "" H 6450 5800 60  0001 C CNN "Comments"
 	1    6450 5800
 	-1   0    0    -1
@@
 P 5150 4200
 F 0 "U7" H 4925 4365 60  0000 C CNN
-F 1 "NP_MOSFET" H 4800 4500 60  0000 C CNN
+F 1 "MOSFET" H 4800 4500 60  0000 C CNN
 F 2 "SOIC8" H 5150 4200 60  0001 C CNN
+F 4 "ROHM" H 5150 4200 60  0001 C CNN "Manufacturer"
+F 5 "SP8M4FU6TB" H 5150 4200 60  0001 C CNN "Mfg. P/N"
+F 6 "1525587" H 5150 4200 60  0001 C CNN "Farnell"
+F 7 "" H 5150 4200 60  0001 C CNN "DigiKey"
+F 8 "" H 5150 4200 60  0001 C CNN "Comments"
 	2    5150 4200
 	1    0    0    1
@@
 P 5150 5800
 F 0 "U7" H 4925 5965 60  0000 C CNN
-F 1 "NP_MOSFET" H 4800 6100 60  0000 C CNN
+F 1 "MOSFET" H 4800 6100 60  0000 C CNN
 F 2 "SOIC8" H 4865 6025 60  0001 C CNN
+F 4 "ROHM" H 5150 5800 60  0001 C CNN "Manufacturer"
+F 5 "SP8M4FU6TB" H 5150 5800 60  0001 C CNN "Mfg. P/N"
+F 6 "1525587" H 5150 5800 60  0001 C CNN "Farnell"
+F 7 "" H 5150 5800 60  0001 C CNN "DigiKey"
+F 8 "" H 5150 5800 60  0001 C CNN "Comments"
 	1    5150 5800
 	1    0    0    -1
 $EndComp
-NoConn ~ 3800 4650
 NoConn ~ 9350 4650
 NoConn ~ 7850 4650
@@
 EN_B
 $Comp
-L GND #PWR024
+L GND #PWR023
 U 1 1 4B8AEABA
 P 2050 6550
-F 0 "#PWR024" H 2050 6550 30  0001 C CNN
+F 0 "#PWR023" H 2050 6550 30  0001 C CNN
 F 1 "GND" H 2050 6480 30  0001 C CNN
 	1    2050 6550
@@
 TODO: R1 and R3 need\nadjustment for V4.\n
 $Comp
-L GND #PWR025
+L GND #PWR024
 U 1 1 4B8A7BF3
 P 4250 2500
-F 0 "#PWR025" H 4250 2500 30  0001 C CNN
+F 0 "#PWR024" H 4250 2500 30  0001 C CNN
 F 1 "GND" H 4250 2430 30  0001 C CNN
 	1    4250 2500
@@
 F 1 "R" H 4500 2150 50  0000 C CNN
 F 2 "SM0402" H 4550 2000 60  0001 C CNN
+F 4 "" H 4400 2100 60  0001 C CNN "Manufacturer"
+F 5 "" H 4400 2100 60  0001 C CNN "Mfg. P/N"
+F 6 "" H 4400 2100 60  0001 C CNN "Farnell"
+F 7 "" H 4400 2100 60  0001 C CNN "DigiKey"
+F 8 "" H 4400 2100 60  0001 C CNN "Comments"
 	1    4400 2100
 	1    0    0    -1
@@
 F 1 "R" V 4700 1800 50  0000 C CNN
 F 2 "SM0402" V 4830 1750 60  0001 C CNN
+F 4 "" H 4700 1800 60  0001 C CNN "Manufacturer"
+F 5 "" H 4700 1800 60  0001 C CNN "Mfg. P/N"
+F 6 "" H 4700 1800 60  0001 C CNN "Farnell"
+F 7 "" H 4700 1800 60  0001 C CNN "DigiKey"
+F 8 "" H 4700 1800 60  0001 C CNN "Comments"
 	1    4700 1800
 	0    1    1    0
 $EndComp
 $Comp
-L GND #PWR026
+L GND #PWR025
 U 1 1 4B8A7A9A
 P 6200 2350
-F 0 "#PWR026" H 6200 2350 30  0001 C CNN
+F 0 "#PWR025" H 6200 2350 30  0001 C CNN
 F 1 "GND" H 6200 2280 30  0001 C CNN
 	1    6200 2350
@@
 $EndComp
 $Comp
-L +BATT #PWR027
+L +BATT #PWR026
 U 1 1 4B8A7A61
 P 5800 1300
-F 0 "#PWR027" H 5800 1250 20  0001 C CNN
+F 0 "#PWR026" H 5800 1250 20  0001 C CNN
 F 1 "+BATT" H 5800 1400 30  0000 C CNN
 	1    5800 1300
@@
 $EndComp
 $Comp
-L +BATT #PWR028
+L +BATT #PWR027
 U 1 1 4B89B9B8
 P 7650 3600
-F 0 "#PWR028" H 7650 3550 20  0001 C CNN
+F 0 "#PWR027" H 7650 3550 20  0001 C CNN
 F 1 "+BATT" H 7650 3700 30  0000 C CNN
 	1    7650 3600
@@
 $EndComp
 $Comp
-L +BATT #PWR029
+L +BATT #PWR028
 U 1 1 4B89B9AA
 P 4000 3600
-F 0 "#PWR029" H 4000 3550 20  0001 C CNN
+F 0 "#PWR028" H 4000 3550 20  0001 C CNN
 F 1 "+BATT" H 4000 3700 30  0000 C CNN
 	1    4000 3600
@@
 $EndComp
 $Comp
-L GND #PWR030
+L GND #PWR029
 U 1 1 4B89B98B
 P 9600 6550
-F 0 "#PWR030" H 9600 6550 30  0001 C CNN
+F 0 "#PWR029" H 9600 6550 30  0001 C CNN
 F 1 "GND" H 9600 6480 30  0001 C CNN
 	1    9600 6550
@@
 $EndComp
 $Comp
-L GND #PWR031
+L GND #PWR030
 U 1 1 4B89B96E
 P 5800 6550
-F 0 "#PWR031" H 5800 6550 30  0001 C CNN
+F 0 "#PWR030" H 5800 6550 30  0001 C CNN
 F 1 "GND" H 5800 6480 30  0001 C CNN
 	1    5800 6550
