File: OpenServo/V4-EDA-preliminary-work/OSv4_H-bridge.sch (KiCad schematic (older format))
At the start: 18 parts, among them M1 CONN_1, M2 CONN_1, M3 CONN_1, U1 ZXCT1009, U5 TC4428A, U6 TC4428A, U7 MOSFET, U8 MOSFET

Commit message: no message
Changed lines of the file:
@@
-EESchema Schematic File Version 2  date 08/05/2010 23:44:42
+EESchema Schematic File Version 2  date 11/05/2010 23:49:02
 LIBS:power
 LIBS:device
@@
 Sheet 3 3
 Title "OpenServo v4 preliminary work-up, © OpenServo project 2010"
-Date "8 may 2010"
+Date "11 may 2010"
 Rev "0.0"
 Comp ""
@@
 	3350 7000 3350 6200
 Wire Wire Line
-	1800 6000 1800 5250
+	1800 5250 1800 6000
 Wire Wire Line
 	1800 6000 2600 6000
 Connection ~ 3900 5250
 Wire Wire Line
-	3900 4650 3900 5250
+	3900 5250 3900 4650
 Wire Wire Line
 	3900 4650 3800 4650
@@
 	6700 4200 7450 4200
 Wire Wire Line
-	6450 6200 6450 6000
+	6450 6000 6450 6200
 Connection ~ 6400 4550
 Wire Wire Line
-	6500 4550 6500 4450
+	6500 4450 6500 4550
 Wire Wire Line
 	6500 4550 6350 4550
@@
 	5100 5450 5100 5550
 Wire Wire Line
-	5150 6200 5150 6000
-Wire Wire Line
-	5100 4550 5100 4450
+	5150 6000 5150 6200
+Wire Wire Line
+	5100 4450 5100 4550
 Wire Wire Line
 	7850 5250 7450 5250
@@
 	4200 5250 4200 5800
 Wire Wire Line
-	3800 2400 3800 2300
+	3800 2300 3800 2400
 Wire Wire Line
 	3800 2400 4400 2400
@@
 	6550 2100 6550 2000
 Wire Wire Line
-	7250 2100 7250 2000
+	7250 2000 7250 2100
 Connection ~ 6900 1500
 Wire Wire Line
@@
 Connection ~ 3800 1800
 Wire Wire Line
-	6200 2100 7250 2100
+	7250 2100 6200 2100
 Connection ~ 5200 5000
 Wire Wire Line
@@
 Connection ~ 5800 6200
 Wire Wire Line
-	6450 6200 5150 6200
+	5150 6200 6450 6200
 Wire Wire Line
 	5150 3800 6450 3800
@@
 Connection ~ 6400 5000
 Wire Wire Line
-	7250 1500 5800 1500
+	5800 1500 7250 1500
 Wire Wire Line
 	5800 1400 5450 1400
@@
 	6450 3800 6450 4000
 Wire Wire Line
-	6350 5450 6350 5550
+	6350 5550 6350 5450
 Wire Wire Line
 	6350 5450 6500 5450
@@
 	4200 4200 4900 4200
 Wire Wire Line
-	3200 5900 3000 5900
-Wire Wire Line
-	3200 6550 3200 5900
+	3000 5900 3200 5900
+Wire Wire Line
+	3200 5900 3200 6550
 Wire Wire Line
 	3350 7000 10100 7000
@@
 Text Notes 1350 4200 0    60   ~ 0
 NOTE: According to the docs, pin 5 on U5 has\n"no internal connection"; it has been used for\nrouting purposes on the PCB.\n\nTODO: TEST!
-Text Notes 900  2650 0    60   ~ 0
+Text Notes 850  3150 0    60   ~ 0
 U5 & U6 (TC4428A): Originally the intention was to use the\nMSOP-8 package which would allow more room on the PCB\nfor other things. However, this packaging only appears to be\navailable when purchased in large quantities; which is not\nworkable for a project where there is an expectation to be\nable to produce low-count runs.
 Text Notes 5200 2550 0    60   ~ 0

Commit message: no message
Parts:
- R1: value R -> 1K; Comments (none) -> 1%, 0.06W; Farnell (none) -> 1358043; Manufacturer (none) -> multicomp; Mfg. P/N (none) -> MC 0.0625W 0402 1% 1K
- R3: value R -> 4.99K; Comments (none) -> 1%, 0.06W; Farnell (none) -> 1803107; Manufacturer (none) -> multicomp; Mfg. P/N (none) -> MC 0.0625W 0402 1% 4K99
- RP2: Comments (none) -> YC124-JR-07100RL is cheaper for lower counts; but footprint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; Farnell 1770152RL -> 1770152
Changed lines of the file:
@@
-EESchema Schematic File Version 2  date 13/05/2010 00:13:19
+EESchema Schematic File Version 2  date 13/05/2010 22:32:29
 LIBS:power
 LIBS:device
@@
 Sheet 3 3
 Title "OpenServo v4 preliminary work-up, © OpenServo project 2010"
-Date "12 may 2010"
+Date "13 may 2010"
 Rev "0.0"
 Comp ""
@@
 F 4 "Bourns" H 2800 6250 60  0001 C CNN "Manufacturer"
 F 5 "CAY10-103J4LF" H 2800 6250 60  0001 C CNN "Mfg. P/N"
-F 6 "1770152RL" H 2800 6250 60  0001 C CNN "Farnell"
+F 6 "1770152" H 2800 6250 60  0001 C CNN "Farnell"
 F 7 "" H 2800 6250 60  0001 C CNN "DigiKey"
-F 8 "" H 2800 6250 60  0001 C CNN "Comments"
+F 8 "YC124-JR-07100RL is cheaper for lower counts; but footprint may need revision" H 2800 6250 60  0001 C CNN "Comments"
 	1    2800 6250
 	1    0    0    -1
@@
 P 4400 2100
 F 0 "R3" H 4500 2050 50  0000 C CNN
-F 1 "R" H 4500 2150 50  0000 C CNN
+F 1 "4.99K" H 4500 2150 50  0000 C CNN
 F 2 "SM0402" H 4550 2000 60  0001 C CNN
-F 4 "" H 4400 2100 60  0001 C CNN "Manufacturer"
-F 5 "" H 4400 2100 60  0001 C CNN "Mfg. P/N"
-F 6 "" H 4400 2100 60  0001 C CNN "Farnell"
+F 4 "multicomp" H 4400 2100 60  0001 C CNN "Manufacturer"
+F 5 "MC 0.0625W 0402 1% 4K99" H 4400 2100 60  0001 C CNN "Mfg. P/N"
+F 6 "1803107" H 4400 2100 60  0001 C CNN "Farnell"
 F 7 "" H 4400 2100 60  0001 C CNN "DigiKey"
-F 8 "" H 4400 2100 60  0001 C CNN "Comments"
+F 8 "1%, 0.06W" H 4400 2100 60  0001 C CNN "Comments"
 	1    4400 2100
 	1    0    0    -1
@@
 U 1 1 4B8A7AF8
 P 4700 1800
-F 0 "R1" V 4780 1800 50  0000 C CNN
-F 1 "R" V 4700 1800 50  0000 C CNN
+F 0 "R1" V 4800 1800 50  0000 C CNN
+F 1 "1K" V 4600 1750 50  0000 C CNN
 F 2 "SM0402" V 4830 1750 60  0001 C CNN
-F 4 "" H 4700 1800 60  0001 C CNN "Manufacturer"
-F 5 "" H 4700 1800 60  0001 C CNN "Mfg. P/N"
-F 6 "" H 4700 1800 60  0001 C CNN "Farnell"
+F 4 "multicomp" H 4700 1800 60  0001 C CNN "Manufacturer"
+F 5 "MC 0.0625W 0402 1% 1K" H 4700 1800 60  0001 C CNN "Mfg. P/N"
+F 6 "1358043" H 4700 1800 60  0001 C CNN "Farnell"
 F 7 "" H 4700 1800 60  0001 C CNN "DigiKey"
-F 8 "" H 4700 1800 60  0001 C CNN "Comments"
+F 8 "1%, 0.06W" H 4700 1800 60  0001 C CNN "Comments"
 	1    4700 1800
 	0    1    1    0
