File: OpenServo/V4-EDA-preliminary-work/OSv4_H-bridge.sch (KiCad schematic (older format))
At the start: 18 parts, among them M1 CONN_1, M2 CONN_1, M3 CONN_1, U1 ZXCT1009, U5 TC4428A, U6 TC4428A, U7 MOSFET, U8 MOSFET

Commit message: no message
Parts:
- RP2: footprint CAY10-XXXJ4 -> CAY16-XXXJ4; Comments YC124-JR-07100RL is cheaper for lower counts; but footprint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 -> (none); Farnell 1770152 -> 1770137; Mfg. P/N CAY10-103J4LF -> CAY16-103J4LF
Changed lines of the file:
@@
-EESchema Schematic File Version 2  date 14/06/2010 08:35:59
+EESchema Schematic File Version 2  date 29/06/2010 00:23:49
 LIBS:power
 LIBS:device
@@
 Sheet 3 3
 Title "OpenServo v4 preliminary work-up, © OpenServo project 2010"
-Date "14 jun 2010"
+Date "28 jun 2010"
 Rev "0.0"
 Comp ""
@@
 F 0 "RP2" H 2800 6700 40  0000 C CNN
 F 1 "R_PACK4" H 2800 6200 40  0000 C CNN
-F 2 "CAY10-XXXJ4" H 2760 6740 60  0001 C CNN
+F 2 "CAY16-XXXJ4" H 2760 6740 60  0001 C CNN
 F 4 "Bourns" H 2800 6250 60  0001 C CNN "Manufacturer"
-F 5 "CAY10-103J4LF" H 2800 6250 60  0001 C CNN "Mfg. P/N"
-F 6 "1770152" H 2800 6250 60  0001 C CNN "Farnell"
+F 5 "CAY16-103J4LF" H 2800 6250 60  0001 C CNN "Mfg. P/N"
+F 6 "1770137" H 2800 6250 60  0001 C CNN "Farnell"
 F 7 "" H 2800 6250 60  0001 C CNN "DigiKey"
-F 8 "YC124-JR-07100RL is cheaper for lower counts; but footprint may need revision" H 2800 6250 60  0001 C CNN "Comments"
+F 8 "" H 2800 6250 60  0001 C CNN "Comments"
 	1    2800 6250
 	1    0    0    -1

Commit message: no message
Parts:
- D2: value 3.6V -> 3.6V Zener; footprint SOD-123 -> SOD-323; symbol ZENER -> ZENER_R; Comments 3.6V, 0.5W, 5% -> 3.6V, 0.2W, 5%; Farnell 1700854 -> 1431199; Manufacturer Fairchild Semiconductor -> On Semiconductor; Mfg. P/N MMSZ5227B -> MM3Z3V6T1G
- U1: footprint SOT23-3 -> SOT23_3
Connections:
- net CURRENT: now also D2.1 (C); no longer D2.2 (K)
- net GND: now also D2.2 (A); no longer D2.1 (A)
Changed lines of the file:
@@
-EESchema Schematic File Version 2  date 29/06/2010 22:50:51
+EESchema Schematic File Version 2  date 02/07/2010 00:00:53
 LIBS:power
 LIBS:device
@@
 Sheet 3 3
 Title "OpenServo v4 preliminary work-up, © OpenServo project 2010"
-Date "29 jun 2010"
+Date "1 jul 2010"
 Rev "0.0"
 Comp ""
@@
 $EndComp
 $Comp
-L ZENER D2
+L ZENER_R D2
 U 1 1 4B9D203D
 P 3800 2100
 F 0 "D2" V 3900 2000 50  0000 C CNN
-F 1 "3.6V" H 3800 2200 40  0000 C CNN
-F 2 "SOD-123" V 3950 1950 60  0001 C CNN
-F 4 "Fairchild Semiconductor" H 3800 2100 60  0001 C CNN "Manufacturer"
-F 5 "MMSZ5227B" H 3800 2100 60  0001 C CNN "Mfg. P/N"
-F 6 "1700854" H 3800 2100 60  0001 C CNN "Farnell"
+F 1 "3.6V Zener" H 3800 2200 40  0000 C CNN
+F 2 "SOD-323" V 3950 1950 60  0001 C CNN
+F 4 "On Semiconductor" H 3800 2100 60  0001 C CNN "Manufacturer"
+F 5 "MM3Z3V6T1G" H 3800 2100 60  0001 C CNN "Mfg. P/N"
+F 6 "1431199" H 3800 2100 60  0001 C CNN "Farnell"
 F 7 "" H 3800 2100 60  0001 C CNN "DigiKey"
-F 8 "3.6V, 0.5W, 5%" H 3800 2100 60  0001 C CNN "Comments"
+F 8 "3.6V, 0.2W, 5%" H 3800 2100 60  0001 C CNN "Comments"
 	1    3800 2100
 	0    -1   -1   0
@@
 F 0 "U1" V 4950 1650 60  0000 C CNN
 F 1 "ZXCT1009" V 5600 1550 60  0000 L CNN
-F 2 "SOT23-3" V 4890 1590 60  0001 C CNN
+F 2 "SOT23_3" V 4890 1590 60  0001 C CNN
 F 4 "Zetex" H 5300 1800 60  0001 C CNN "Manufacturer"
 F 5 "ZXCT1009FTA" H 5300 1800 60  0001 C CNN "Mfg. P/N"
