File: OpenServo/V4-EDA-preliminary-work/OSv4_logic.sch (KiCad schematic (older format))
At the start: 36 parts, among them P1-1 P1, P1-10 P1, P1-2 P1, P1-3 P1, P1-4 P1, P1-5 P1, P1-6 P1, P1-7 P1, P1-8 P1, P1-9 P1, U2 MCP9701A, U3 LM3480IM-3.3, U4 ATXMEGA32A4

Commit message: no message
Parts:
- renumbered C13 to C10, C14 to C11, C17 to C12, C18 to C13, C11 to C8, C12 to C9, JP9 to JP4, JP11 to JP5
Changed lines of the file:
@@
-EESchema Schematic File Version 2  date 25/04/2010 17:16:50
+EESchema Schematic File Version 2  date 04/05/2010 11:09:49
 LIBS:power
 LIBS:device
@@
 Sheet 2 3
 Title "OpenServo v4 preliminary work-up, © OpenServo project 2010"
-Date "25 apr 2010"
+Date "4 may 2010"
 Rev "0.0"
 Comp ""
@@
 	7750 6850 7750 4000
 $Comp
-L OPTION JP11
+L OPTION JP5
 U 1 1 4B8AE5FB
 P 6250 3800
-F 0 "JP11" H 6300 3800 60  0000 C CNN
+F 0 "JP5" H 6300 3800 60  0000 C CNN
 F 1 "+3.3V" H 6525 3800 40  0000 C CNN
 F 2 "OPTPAD" H 6250 3800 60  0001 C CNN
@@
 EN_B
 $Comp
-L CP1 C18
+L CP1 C13
 U 1 1 4B96CAE1
 P 10400 6100
-F 0 "C18" H 10450 6200 50  0000 L CNN
+F 0 "C13" H 10450 6200 50  0000 L CNN
 F 1 "33uF 4V" H 10450 6000 50  0000 L CNN
 F 2 "SM0603" H 10500 6250 60  0001 C CNN
@@
 $EndComp
 $Comp
-L OPTION JP9
+L OPTION JP4
 U 1 1 4B8AE5C3
 P 6250 4000
-F 0 "JP9" H 6275 4000 60  0000 C CNN
+F 0 "JP4" H 6275 4000 60  0000 C CNN
 F 1 "PB2" H 6475 4000 40  0000 C CNN
 F 2 "OPTPAD" H 6250 4000 60  0001 C CNN
@@
 NOTE: Decoupling capacitors to be placed close to the device for each supply pin pair in a signal group.
 $Comp
-L C C14
+L C C11
 U 1 1 4B8A9346
 P 1450 5500
-F 0 "C14" V 1500 5375 50  0000 L CNN
+F 0 "C11" V 1500 5375 50  0000 L CNN
 F 1 "100nF" V 1500 5675 50  0000 L CNN
 F 2 "SM0402" V 1550 5325 60  0001 C CNN
@@
 $EndComp
 $Comp
-L C C13
+L C C10
 U 1 1 4B8A9340
 P 1450 5100
-F 0 "C13" V 1500 4975 50  0000 L CNN
+F 0 "C10" V 1500 4975 50  0000 L CNN
 F 1 "100nF" V 1500 5275 50  0000 L CNN
 F 2 "SM0402" V 1550 4925 60  0001 C CNN
@@
 $EndComp
 $Comp
-L C C12
+L C C9
 U 1 1 4B8A92EF
 P 1450 4700
-F 0 "C12" V 1500 4575 50  0000 L CNN
+F 0 "C9" V 1500 4575 50  0000 L CNN
 F 1 "100nF" V 1500 4875 50  0000 L CNN
 F 2 "SM0402" V 1550 4525 60  0001 C CNN
@@
 $EndComp
 $Comp
-L C C11
+L C C8
 U 1 1 4B8A8D44
 P 1450 4300
-F 0 "C11" V 1500 4175 50  0000 L CNN
+F 0 "C8" V 1500 4175 50  0000 L CNN
 F 1 "100nF" V 1500 4475 50  0000 L CNN
 F 2 "SM0402" H 1450 4300 60  0001 C CNN
@@
 $EndComp
 $Comp
-L CP1 C17
+L CP1 C12
 U 1 1 4B86F81A
 P 8800 6100
-F 0 "C17" H 8850 6200 50  0000 L CNN
+F 0 "C12" H 8850 6200 50  0000 L CNN
 F 1 "47uF 16V" H 8850 6000 50  0000 L CNN
 F 2 "SM0603" H 8900 6250 60  0001 C CNN

Commit message: no message
Parts:
- removed L2: 47nH, 5%, DCR<0.3ohm, >100mA, SM0603, symbol INDUCTOR
- C10, C11, C8, C9: value 100nF -> 0.1uF
- L1: value INDUCTOR -> 10uH; footprint SM0603 -> MLF1608E100K; Comments (none) -> 10%, Max DC R 1.7ohm, 10ma; DigiKey (none) -> 445-1025-1-ND; Farnell (none) -> 1669541; Manufacturer (none) -> TDK; Mfg. P/N (none) -> MLF1608E100K
- P1-1: Comments (none) -> Part numbers for Tin - Gold: DF11-10DP-2DSA(01), H2853-ND; DigiKey (none) -> H10232-ND; Manufacturer (none) -> Hirose; Mfg. P/N (none) -> DF11-10DP-2DSA(24)
- R4: Comments (none) -> 1%, 0.06W; Farnell (none) -> 1358082; Manufacturer (none) -> multicomp; Mfg. P/N (none) -> MC 0.0625W 0402 1% 10K
- R5: renamed from R6; Comments (none) -> 1%, 0.06W; Farnell (none) -> 1358069; Manufacturer (none) -> multicomp; Mfg. P/N (none) -> MC 0.0625W 0402 1% 10K
- RP1: Farnell (none) -> 1770149RL; Manufacturer (none) -> Bourns; Mfg. P/N (none) -> CAY10-101J4LF
- U2: footprint SOT23_3 -> SOT23-3; DigiKey (none) -> MCP9701AT-E/TTCT-ND; Manufacturer (none) -> Microchip; Mfg. P/N (none) -> MCP9701AT-E/TT
- U3: footprint SOT23_3 -> SOT23-3; DigiKey (none) -> LM3480IM3-3.3CT-ND; Farnell (none) -> 1469102; Manufacturer (none) -> National Semiconductor; Mfg. P/N (none) -> LM3480IM3-3.3/NOPB
- U4: Comments (none) -> Also consider: ATXMEGA32D4 (DigiKey: ATXMEGA32D4-MH-ND); Manufacturer (none) -> Atmel; Mfg. P/N (none) -> ATxmega32A4-MH
- renumbered R19 to R6
Connections:
- wire segments 134 -> 133
Other:
- note added: "47nH, 5%, DCR<0.3ohm, >100mA"
- note added: "C12 and C13 are to be\nplaced close to U3\n"
- note added: "One might use an inductor\nbetween vcc and C13; but\nthe cramped noisy nature\nof the OS PCB means that\nit is likely not overly useful\nand merely wastes space?"
- note added: "R4 and R5 are\nscaled for a\nmaximum of 12V\n(BATTV=3V @ 12V)\n"
- note removed: "C17 and C18 are to be\nplaced close to U3\n"
- note removed: "R4 and R6 are\nscaled for a\nmaximum of 12V\n(BATTV=3V @ 12V)\n"

Commit message: no message
Parts:
- C10, C11, C6, C7, C8, C9: Comments (none) -> X7R, ±10%, 16V, Ceramic; Farnell (none) -> 1758896; Manufacturer (none) -> multicomp; Mfg. P/N (none) -> MCCA000050
- C12: value 47uF 16V -> 22uF 16V; Comments (none) -> Maybe TR3B226K016C0600 if smaller physical size is needed; Farnell (none) -> 1754088; Manufacturer (none) -> Vishay Sprague; Mfg. P/N (none) -> TR3C226K016C0375
- C13: value 33uF 4V -> 4.7uF 16V; footprint SM0603 -> SM0402; Farnell (none) -> 1754083; Manufacturer (none) -> Vishay Sprague; Mfg. P/N (none) -> TR3A475K016C2000
- D1: footprint SM0402 -> SOD-923; Comments (none) -> IF 100mA; Farnell (none) -> 1453608; Manufacturer (none) -> On Semiconductor; Mfg. P/N (none) -> NSR0130P2T5G
- R6: Comments (none) -> 1%, 0.06W; Farnell (none) -> 1358069; Manufacturer (none) -> multicomp; Mfg. P/N (none) -> MC 0.0625W 0402 1% 10K
- RP1: footprint RP0804 -> CAY10-XXXJ4
Other:
- note removed: "Brown-out protection\nOptional? (no) Value?"
Changed lines of the file:
@@
-EESchema Schematic File Version 2  date 07/05/2010 17:07:47
+EESchema Schematic File Version 2  date 08/05/2010 00:59:33
 LIBS:power
 LIBS:device
@@
 F 0 "RP1" H 6250 2150 40  0000 C CNN
 F 1 "R_PACK4" H 6250 1650 40  0000 C CNN
-F 2 "RP0804" H 6210 2190 60  0001 C CNN
+F 2 "CAY10-XXXJ4" H 6210 2190 60  0001 C CNN
 F 4 "Bourns" H 6250 1700 60  0001 C CNN "Manufacturer"
 F 5 "CAY10-101J4LF" H 6250 1700 60  0001 C CNN "Mfg. P/N"
@@
 Text Notes 5950 2250 0    60   Italic 0
 optional?
-Text Notes 8900 5400 0    60   Italic 0
-Brown-out protection\nOptional? (no) Value?
 $Comp
 L OPTION JP3
@@
 P 10400 6100
 F 0 "C13" H 10450 6200 50  0000 L CNN
-F 1 "33uF 4V" H 10450 6000 50  0000 L CNN
-F 2 "SM0603" H 10500 6250 60  0001 C CNN
+F 1 "4.7uF 16V" H 10450 6000 50  0000 L CNN
+F 2 "SM0402" H 10500 6250 60  0001 C CNN
+F 4 "Vishay Sprague" H 10400 6100 60  0001 C CNN "Manufacturer"
+F 5 "TR3A475K016C2000" H 10400 6100 60  0001 C CNN "Mfg. P/N"
+F 6 "1754083" H 10400 6100 60  0001 C CNN "Farnell"
+F 7 "" H 10400 6100 60  0001 C CNN "DigiKey"
+F 8 "" H 10400 6100 60  0001 C CNN "Comments"
 	1    10400 6100
 	1    0    0    -1
@@
 F 1 "0.1uF" V 1500 5675 50  0000 L CNN
 F 2 "SM0402" V 1550 5325 60  0001 C CNN
+F 4 "multicomp" H 1450 5500 60  0001 C CNN "Manufacturer"
+F 5 "MCCA000050" H 1450 5500 60  0001 C CNN "Mfg. P/N"
+F 6 "1758896" H 1450 5500 60  0001 C CNN "Farnell"
+F 7 "" H 1450 5500 60  0001 C CNN "DigiKey"
+F 8 "X7R, ±10%, 16V, Ceramic" H 1450 5500 60  0001 C CNN "Comments"
 	1    1450 5500
 	0    1    1    0
@@
 F 1 "0.1uF" V 1500 5275 50  0000 L CNN
 F 2 "SM0402" V 1550 4925 60  0001 C CNN
+F 4 "multicomp" H 1450 5100 60  0001 C CNN "Manufacturer"
+F 5 "MCCA000050" H 1450 5100 60  0001 C CNN "Mfg. P/N"
+F 6 "1758896" H 1450 5100 60  0001 C CNN "Farnell"
+F 7 "" H 1450 5100 60  0001 C CNN "DigiKey"
+F 8 "X7R, ±10%, 16V, Ceramic" H 1450 5100 60  0001 C CNN "Comments"
 	1    1450 5100
 	0    1    1    0
@@
 F 1 "0.1uF" V 1500 4875 50  0000 L CNN
 F 2 "SM0402" V 1550 4525 60  0001 C CNN
+F 4 "multicomp" H 1450 4700 60  0001 C CNN "Manufacturer"
+F 5 "MCCA000050" H 1450 4700 60  0001 C CNN "Mfg. P/N"
+F 6 "1758896" H 1450 4700 60  0001 C CNN "Farnell"
+F 7 "" H 1450 4700 60  0001 C CNN "DigiKey"
+F 8 "X7R, ±10%, 16V, Ceramic" H 1450 4700 60  0001 C CNN "Comments"
 	1    1450 4700
 	0    1    1    0
@@
 F 1 "10.0K" H 1950 3200 50  0000 C CNN
 F 2 "SM0402" H 1750 3150 60  0001 C CNN
+F 4 "multicomp" H 1750 3150 60  0001 C CNN "Manufacturer"
+F 5 "MC 0.0625W 0402 1% 10K" H 1750 3150 60  0001 C CNN "Mfg. P/N"
+F 6 "1358069" H 1750 3150 60  0001 C CNN "Farnell"
+F 7 "" H 1750 3150 60  0001 C CNN "DigiKey"
+F 8 "1%, 0.06W" H 1750 3150 60  0001 C CNN "Comments"
 	1    1750 3150
 	1    0    0    -1
@@
 F 1 "0.1uF" V 1500 4475 50  0000 L CNN
 F 2 "SM0402" H 1450 4300 60  0001 C CNN
+F 4 "multicomp" H 1450 4300 60  0001 C CNN "Manufacturer"
+F 5 "MCCA000050" H 1450 4300 60  0001 C CNN "Mfg. P/N"
+F 6 "1758896" H 1450 4300 60  0001 C CNN "Farnell"
+F 7 "" H 1450 4300 60  0001 C CNN "DigiKey"
+F 8 "X7R, ±10%, 16V, Ceramic" H 1450 4300 60  0001 C CNN "Comments"
 	1    1450 4300
 	0    1    1    0
@@
 F 0 "D1" V 8800 5700 40  0000 C CNN
 F 1 "DIODE" H 8800 5500 40  0000 C CNN
-F 2 "SM0402" V 8760 5740 60  0001 C CNN
+F 2 "SOD-923" V 8760 5740 60  0001 C CNN
+F 4 "On Semiconductor" H 8800 5600 60  0001 C CNN "Manufacturer"
+F 5 "NSR0130P2T5G" H 8800 5600 60  0001 C CNN "Mfg. P/N"
+F 6 "1453608" H 8800 5600 60  0001 C CNN "Farnell"
+F 7 "" H 8800 5600 60  0001 C CNN "DigiKey"
+F 8 "IF 100mA" H 8800 5600 60  0001 C CNN "Comments"
 	1    8800 5600
 	0    1    1    0
@@
 P 8800 6100
 F 0 "C12" H 8850 6200 50  0000 L CNN
-F 1 "47uF 16V" H 8850 6000 50  0000 L CNN
+F 1 "22uF 16V" H 8850 6000 50  0000 L CNN
 F 2 "SM0603" H 8900 6250 60  0001 C CNN
+F 4 "Vishay Sprague" H 8800 6100 60  0001 C CNN "Manufacturer"
+F 5 "TR3C226K016C0375" H 8800 6100 60  0001 C CNN "Mfg. P/N"
+F 6 "1754088" H 8800 6100 60  0001 C CNN "Farnell"
+F 7 "" H 8800 6100 60  0001 C CNN "DigiKey"
+F 8 "Maybe TR3B226K016C0600 if smaller physical size is needed" H 8800 6100 60  0001 C CNN "Comments"
 	1    8800 6100
 	1    0    0    -1
@@
 F 1 "0.1uF" H 10550 1600 50  0000 L CNN
 F 2 "SM0402" H 10600 1850 60  0001 C CNN
+F 4 "multicomp" H 10500 1700 60  0001 C CNN "Manufacturer"
+F 5 "MCCA000050" H 10500 1700 60  0001 C CNN "Mfg. P/N"
+F 6 "1758896" H 10500 1700 60  0001 C CNN "Farnell"
+F 7 "" H 10500 1700 60  0001 C CNN "DigiKey"
+F 8 "X7R, ±10%, 16V, Ceramic" H 10500 1700 60  0001 C CNN "Comments"
 	1    10500 1700
 	1    0    0    -1
@@
 F 1 "0.1uF" H 2800 1900 50  0000 L CNN
 F 2 "SM0402" H 2850 2150 60  0001 C CNN
+F 4 "multicomp" H 2750 2000 60  0001 C CNN "Manufacturer"
+F 5 "MCCA000050" H 2750 2000 60  0001 C CNN "Mfg. P/N"
+F 6 "1758896" H 2750 2000 60  0001 C CNN "Farnell"
+F 7 "" H 2750 2000 60  0001 C CNN "DigiKey"
+F 8 "X7R, ±10%, 16V, Ceramic" H 2750 2000 60  0001 C CNN "Comments"
 	1    2750 2000
 	1    0    0    -1

Commit message: no message
Connections:
- wire segments 133 -> 129
- no-connect marks 10 -> 19
Other:
- note added: "RP1"
- note added: "RP1 would have provided some limited protection against\nconnection and programming errors; however design\nconsiderations on the PCB mean that this is one of the\nitems that probably has to be dropped from the design."
- note removed: "optional?"
- moved on the sheet: RP1
