File: OpenServo/V4-EDA-preliminary-work/OSv4_logic.sch (KiCad schematic (older format))
At the start: 35 parts, among them P1-1 P1, P1-10 P1, P1-2 P1, P1-3 P1, P1-4 P1, P1-5 P1, P1-6 P1, P1-7 P1, P1-8 P1, P1-9 P1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

Commit message: no message
Other:
- note added: "NOTE: The XMEGA has an integrated temperature sensor.\nHowever, U2 can be placed close to the MOSFETs and\nmotor end of the PCB; which likely gives more qualitative\ndata than using the one inside the MCU. Could U2 be\ndropped if board space becomes a problem?"
- note added: "RP1 would have provided some limited protection against\nconnection and programming errors; however design\nconsiderations on the PCB mean that this is one of the\nitems that probably has to be dropped."
- note removed: "RP1 would have provided some limited protection against\nconnection and programming errors; however design\nconsiderations on the PCB mean that this is one of the\nitems that probably has to be dropped from the design."

Commit message: no message
Parts:
- D1: symbol DIODE -> DIODE2
Changed lines of the file:
@@
-EESchema Schematic File Version 2  date 11/05/2010 23:49:02
+EESchema Schematic File Version 2  date 13/05/2010 00:13:19
 LIBS:power
 LIBS:device
@@
 Sheet 2 3
 Title "OpenServo v4 preliminary work-up, © OpenServo project 2010"
-Date "11 may 2010"
+Date "12 may 2010"
 Rev "0.0"
 Comp ""
@@
 $EndComp
 $Comp
-L DIODE D1
+L DIODE2 D1
 U 1 1 4B86F84F
 P 8800 5600

Commit message: no message
Parts:
- RP1: Farnell 1770149RL -> 1770149
Changed lines of the file:
@@
-EESchema Schematic File Version 2  date 13/05/2010 00:13:19
+EESchema Schematic File Version 2  date 13/05/2010 22:32:29
 LIBS:power
 LIBS:device
@@
 Sheet 2 3
 Title "OpenServo v4 preliminary work-up, © OpenServo project 2010"
-Date "12 may 2010"
+Date "13 may 2010"
 Rev "0.0"
 Comp ""
@@
 F 4 "Bourns" H 7800 2200 60  0001 C CNN "Manufacturer"
 F 5 "CAY10-101J4LF" H 7800 2200 60  0001 C CNN "Mfg. P/N"
-F 6 "1770149RL" H 7800 2200 60  0001 C CNN "Farnell"
+F 6 "1770149" H 7800 2200 60  0001 C CNN "Farnell"
 F 7 "" H 7800 2200 60  0001 C CNN "DigiKey"
 F 8 "" H 7800 2200 60  0001 C CNN "Comments"
