File: OpenServo/V4-EDA-preliminary-work/OSv4_logic.sch (KiCad schematic (older format))
At the start: 35 parts, among them P1-1 P1, P1-10 P1, P1-2 P1, P1-3 P1, P1-4 P1, P1-5 P1, P1-6 P1, P1-7 P1, P1-8 P1, P1-9 P1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

Commit message: no message
Parts:
- removed C13: 4.7uF 16V, SM0402, symbol CP1
- C12: value 22uF 16V -> 10uF 16V; footprint SM0603 -> SMC3216; Comments Maybe TR3B226K016C0600 if smaller physical size is needed -> (none); Farnell 1754088 -> 1754086; Mfg. P/N TR3C226K016C0375 -> TR3A106K016C1700
Other:
- note added: "C13,4.7uF 16V,SMC3216\nTR3A475K016C2000"
Changed lines of the file:
@@
-EESchema Schematic File Version 2  date 15/05/2010 00:33:24
+EESchema Schematic File Version 2  date 14/06/2010 08:35:59
 LIBS:power
 LIBS:device
@@
 Sheet 2 3
 Title "OpenServo v4 preliminary work-up, © OpenServo project 2010"
-Date "14 may 2010"
+Date "14 jun 2010"
 Rev "0.0"
 Comp ""
@@
 Comment4 ""
 $EndDescr
-Text Notes 2100 2600 0    60   ~ 0
-NOTE: The XMEGA has an integrated temperature sensor.\nHowever, U2 can be placed close to the MOSFETs and\nmotor end of the PCB; which likely gives more qualitative\ndata than using the one inside the MCU. Could U2 be\ndropped if board space becomes a problem?
+Wire Wire Line
+	10400 4950 10400 5900
+Wire Wire Line
+	10400 6450 10400 6300
+Text Notes 11100 6100 2    39   Italic 0
+C13,4.7uF 16V,SMC3216\nTR3A475K016C2000
 Connection ~ 6850 2050
 Wire Wire Line
@@
 Connection ~ 6550 1950
 Wire Wire Line
-	6550 1950 6550 2450
+	6550 2450 6550 1950
 Wire Wire Line
 	5350 1850 7050 1850
@@
 Connection ~ 10400 5650
 Wire Wire Line
-	10400 5900 10400 4950
-Wire Wire Line
 	6650 2350 7050 2350
 Wire Wire Line
@@
 	6200 6250 4500 6250
 Wire Wire Line
-	10400 6450 10400 6300
-Wire Wire Line
 	9600 6350 9600 6650
 Wire Wire Line
@@
 	2750 2200 1250 2200
 Wire Wire Line
-	1400 1650 1250 1650
-Wire Wire Line
-	1250 1650 1250 2400
+	1250 1650 1400 1650
+Wire Wire Line
+	1250 2400 1250 1650
 Wire Wire Line
 	1400 1800 800  1800
@@
 Connection ~ 1700 4700
 Wire Wire Line
-	1700 4550 850  4550
+	850  4550 1700 4550
 Wire Wire Line
 	1700 5100 1700 4950
@@
 Connection ~ 1700 5500
 Wire Wire Line
-	1700 5350 850  5350
-Wire Wire Line
-	850  5350 850  2800
+	850  5350 1700 5350
+Wire Wire Line
+	850  2800 850  5350
 Connection ~ 850  4950
 Wire Wire Line
@@
 Connection ~ 1050 5100
 Wire Wire Line
-	1250 4300 1050 4300
-Wire Wire Line
-	1050 4300 1050 5850
+	1050 4300 1250 4300
+Wire Wire Line
+	1050 5850 1050 4300
 Connection ~ 1050 4500
 Wire Wire Line
@@
 	5110 2100 4890 2100
 Wire Wire Line
-	9850 1850 10100 1850
-Wire Wire Line
-	10100 1850 10100 2350
+	10100 1850 9850 1850
+Wire Wire Line
+	10100 2350 10100 1850
 Wire Wire Line
 	5950 1750 5950 1550
@@
 Wire Wire Line
 	6750 2250 6750 1750
+Wire Notes Line
+	10500 5950 10300 5950
+Wire Notes Line
+	10500 5950 10500 6250
+Wire Notes Line
+	10500 6250 10300 6250
+Wire Notes Line
+	10300 6250 10300 5950
+Connection ~ 10400 6300
+Connection ~ 10400 5900
+Text Notes 2100 2600 0    60   ~ 0
+NOTE: The XMEGA has an integrated temperature sensor.\nHowever, U2 can be placed close to the MOSFETs and\nmotor end of the PCB; which likely gives more qualitative\ndata than using the one inside the MCU. Could U2 be\ndropped if board space becomes a problem?
 NoConn ~ 8000 2250
 NoConn ~ 8000 2350
@@
 Text GLabel 6450 6150 2    60   Output ~ 0
 EN_B
-$Comp
-L CP1 C13
-U 1 1 4B96CAE1
-P 10400 6100
-F 0 "C13" H 10450 6200 50  0000 L CNN
-F 1 "4.7uF 16V" H 10450 6000 50  0000 L CNN
-F 2 "SM0402" H 10500 6250 60  0001 C CNN
-F 4 "Vishay Sprague" H 10400 6100 60  0001 C CNN "Manufacturer"
-F 5 "TR3A475K016C2000" H 10400 6100 60  0001 C CNN "Mfg. P/N"
-F 6 "1754083" H 10400 6100 60  0001 C CNN "Farnell"
-F 7 "" H 10400 6100 60  0001 C CNN "DigiKey"
-F 8 "" H 10400 6100 60  0001 C CNN "Comments"
-	1    10400 6100
-	1    0    0    -1
-$EndComp
 Text Label 7050 1450 0    30   ~ 0
 PA7_(GPIO)
@@
 P 8800 6100
 F 0 "C12" H 8850 6200 50  0000 L CNN
-F 1 "22uF 16V" H 8850 6000 50  0000 L CNN
-F 2 "SM0603" H 8900 6250 60  0001 C CNN
+F 1 "10uF 16V" H 8850 6000 50  0000 L CNN
+F 2 "SMC3216" H 8900 6250 60  0001 C CNN
 F 4 "Vishay Sprague" H 8800 6100 60  0001 C CNN "Manufacturer"
-F 5 "TR3C226K016C0375" H 8800 6100 60  0001 C CNN "Mfg. P/N"
-F 6 "1754088" H 8800 6100 60  0001 C CNN "Farnell"
+F 5 "TR3A106K016C1700" H 8800 6100 60  0001 C CNN "Mfg. P/N"
+F 6 "1754086" H 8800 6100 60  0001 C CNN "Farnell"
 F 7 "" H 8800 6100 60  0001 C CNN "DigiKey"
-F 8 "Maybe TR3B226K016C0600 if smaller physical size is needed" H 8800 6100 60  0001 C CNN "Comments"
+F 8 "" H 8800 6100 60  0001 C CNN "Comments"
 	1    8800 6100
 	1    0    0    -1

Commit message: no message
Parts:
- C6: footprint SM0402 -> SM0603; Farnell 1758896 -> 9406140; Mfg. P/N MCCA000050 -> B0603R104KCT
Changed lines of the file:
@@
-EESchema Schematic File Version 2  date 14/06/2010 08:35:59
+EESchema Schematic File Version 2  date 29/06/2010 00:23:49
 LIBS:power
 LIBS:device
@@
 Sheet 2 3
 Title "OpenServo v4 preliminary work-up, © OpenServo project 2010"
-Date "14 jun 2010"
+Date "28 jun 2010"
 Rev "0.0"
 Comp ""
@@
 F 0 "C6" H 10550 1800 50  0000 L CNN
 F 1 "0.1uF" H 10550 1600 50  0000 L CNN
-F 2 "SM0402" H 10600 1850 60  0001 C CNN
+F 2 "SM0603" H 10600 1850 60  0001 C CNN
 F 4 "multicomp" H 10500 1700 60  0001 C CNN "Manufacturer"
-F 5 "MCCA000050" H 10500 1700 60  0001 C CNN "Mfg. P/N"
-F 6 "1758896" H 10500 1700 60  0001 C CNN "Farnell"
+F 5 "B0603R104KCT" H 10500 1700 60  0001 C CNN "Mfg. P/N"
+F 6 "9406140" H 10500 1700 60  0001 C CNN "Farnell"
 F 7 "" H 10500 1700 60  0001 C CNN "DigiKey"
 F 8 "X7R, ±10%, 16V, Ceramic" H 10500 1700 60  0001 C CNN "Comments"

Commit message: no message
Parts:
- C6: footprint SM0603 -> SM0402; Farnell 9406140 -> 1758896; Mfg. P/N B0603R104KCT -> MCCA000050
Changed lines of the file:
@@
-EESchema Schematic File Version 2  date 29/06/2010 00:23:49
+EESchema Schematic File Version 2  date 29/06/2010 22:50:51
 LIBS:power
 LIBS:device
@@
 Sheet 2 3
 Title "OpenServo v4 preliminary work-up, © OpenServo project 2010"
-Date "28 jun 2010"
+Date "29 jun 2010"
 Rev "0.0"
 Comp ""
@@
 F 0 "C6" H 10550 1800 50  0000 L CNN
 F 1 "0.1uF" H 10550 1600 50  0000 L CNN
-F 2 "SM0603" H 10600 1850 60  0001 C CNN
+F 2 "SM0402" H 10600 1850 60  0001 C CNN
 F 4 "multicomp" H 10500 1700 60  0001 C CNN "Manufacturer"
-F 5 "B0603R104KCT" H 10500 1700 60  0001 C CNN "Mfg. P/N"
-F 6 "9406140" H 10500 1700 60  0001 C CNN "Farnell"
+F 5 "MCCA000050" H 10500 1700 60  0001 C CNN "Mfg. P/N"
+F 6 "1758896" H 10500 1700 60  0001 C CNN "Farnell"
 F 7 "" H 10500 1700 60  0001 C CNN "DigiKey"
 F 8 "X7R, ±10%, 16V, Ceramic" H 10500 1700 60  0001 C CNN "Comments"

Commit message: no message
Parts:
- RP1: footprint CAY10-XXXJ4 -> CAY16-XXXJ4; Farnell 1770149 -> 1770131; Mfg. P/N CAY10-101J4LF -> CAY16-101J4LF
- U2, U3: footprint SOT23-3 -> SOT23_3
Changed lines of the file:
@@
-EESchema Schematic File Version 2  date 29/06/2010 22:50:51
+EESchema Schematic File Version 2  date 02/07/2010 00:00:53
 LIBS:power
 LIBS:device
@@
 Sheet 2 3
 Title "OpenServo v4 preliminary work-up, © OpenServo project 2010"
-Date "29 jun 2010"
+Date "1 jul 2010"
 Rev "0.0"
 Comp ""
@@
 	10400 4950 10400 5900
 Wire Wire Line
-	10400 6450 10400 6300
+	10400 6300 10400 6450
 Text Notes 11100 6100 2    39   Italic 0
 C13,4.7uF 16V,SMC3216\nTR3A475K016C2000
@@
 Connection ~ 6550 1950
 Wire Wire Line
-	6550 2450 6550 1950
+	6550 1950 6550 2450
 Wire Wire Line
 	5350 1850 7050 1850
@@
 Connection ~ 8800 6450
 Wire Wire Line
-	8400 6450 10400 6450
+	10400 6450 8400 6450
 Connection ~ 1750 4300
 Wire Wire Line
@@
 	2750 2200 1250 2200
 Wire Wire Line
-	1250 1650 1400 1650
-Wire Wire Line
-	1250 2400 1250 1650
+	1400 1650 1250 1650
+Wire Wire Line
+	1250 1650 1250 2400
 Wire Wire Line
 	1400 1800 800  1800
@@
 Connection ~ 1700 4700
 Wire Wire Line
-	850  4550 1700 4550
+	1700 4550 850  4550
 Wire Wire Line
 	1700 5100 1700 4950
@@
 Connection ~ 1700 5500
 Wire Wire Line
-	850  5350 1700 5350
-Wire Wire Line
-	850  2800 850  5350
+	1700 5350 850  5350
+Wire Wire Line
+	850  5350 850  2800
 Connection ~ 850  4950
 Wire Wire Line
@@
 Connection ~ 1050 5100
 Wire Wire Line
-	1050 4300 1250 4300
-Wire Wire Line
-	1050 5850 1050 4300
+	1250 4300 1050 4300
+Wire Wire Line
+	1050 4300 1050 5850
 Connection ~ 1050 4500
 Wire Wire Line
@@
 	5110 2100 4890 2100
 Wire Wire Line
-	10100 1850 9850 1850
-Wire Wire Line
-	10100 2350 10100 1850
+	9850 1850 10100 1850
+Wire Wire Line
+	10100 1850 10100 2350
 Wire Wire Line
 	5950 1750 5950 1550
@@
 F 0 "U2" H 1700 2000 60  0000 L CNN
 F 1 "MCP9701A" H 2200 1500 60  0000 R CNN
-F 2 "SOT23-3" H 1640 2060 60  0001 C CNN
+F 2 "SOT23_3" H 1640 2060 60  0001 C CNN
 F 4 "Microchip" H 2200 1750 60  0001 C CNN "Manufacturer"
 F 5 "MCP9701AT-E/TT" H 2200 1750 60  0001 C CNN "Mfg. P/N"
@@
 F 0 "RP1" H 7800 2650 40  0000 C CNN
 F 1 "R_PACK4" H 7800 2150 40  0000 C CNN
-F 2 "CAY10-XXXJ4" H 7760 2690 60  0001 C CNN
+F 2 "CAY16-XXXJ4" H 7760 2690 60  0001 C CNN
 F 4 "Bourns" H 7800 2200 60  0001 C CNN "Manufacturer"
-F 5 "CAY10-101J4LF" H 7800 2200 60  0001 C CNN "Mfg. P/N"
-F 6 "1770149" H 7800 2200 60  0001 C CNN "Farnell"
+F 5 "CAY16-101J4LF" H 7800 2200 60  0001 C CNN "Mfg. P/N"
+F 6 "1770131" H 7800 2200 60  0001 C CNN "Farnell"
 F 7 "" H 7800 2200 60  0001 C CNN "DigiKey"
 F 8 "" H 7800 2200 60  0001 C CNN "Comments"
@@
 F 0 "U3" H 9425 6325 60  0000 C CNN
 F 1 "LM3480IM-3.3" H 9650 5725 60  0000 L CNN
-F 2 "SOT23-3" H 9365 6385 60  0001 C CNN
+F 2 "SOT23_3" H 9365 6385 60  0001 C CNN
 F 4 "National Semiconductor" H 9600 6000 60  0001 C CNN "Manufacturer"
 F 5 "LM3480IM3-3.3/NOPB" H 9600 6000 60  0001 C CNN "Mfg. P/N"

Commit message: no message
Parts:
- L1: Comments 10%, Max DC R 1.7ohm, 10ma -> 10%, Max DC R 1.7ohm, 10ma, magnetic shielded
Changed lines of the file:
@@
-EESchema Schematic File Version 2  date 02/07/2010 00:00:53
+EESchema Schematic File Version 2  date 04/07/2010 10:22:34
 LIBS:power
 LIBS:device
@@
 Sheet 2 3
 Title "OpenServo v4 preliminary work-up, © OpenServo project 2010"
-Date "1 jul 2010"
+Date "4 jul 2010"
 Rev "0.0"
 Comp ""
@@
 F 6 "1669541" H 1300 4050 60  0001 C CNN "Farnell"
 F 7 "445-1025-1-ND" H 1300 4050 60  0001 C CNN "DigiKey"
-F 8 "10%, Max DC R 1.7ohm, 10ma" H 1300 4050 60  0001 C CNN "Comments"
+F 8 "10%, Max DC R 1.7ohm, 10ma, magnetic shielded" H 1300 4050 60  0001 C CNN "Comments"
 	1    1300 4050
 	0    -1   -1   0

Commit message: no message
Other:
- note added: "R5 - servo pot\noff board"
- note removed: "R5 - serbo pot\noff board"
Changed lines of the file:
@@
-EESchema Schematic File Version 2  date 04/07/2010 10:22:34
+EESchema Schematic File Version 2  date 04/07/2010 23:28:30
 LIBS:power
 LIBS:device
@@
 NoConn ~ 1850 6050
 Text Notes 9200 1350 0    60   ~ 0
-R5 - serbo pot\noff board
+R5 - servo pot\noff board
 $Comp
 L CONN_1 POT3
